Commit message: update test

File: tests/sample/robot.urdf (robot description, URDF)
Before this commit: robot robot, 20 links, 19 joints
Joints:
- joint L_ankle_y: limit lower=-0.698 upper=0.698 effort=17 velocity=0 -> lower=-0.698 upper=0.698 effort=17 velocity=10
- joint L_elbow_x: type revolute -> fixed
- joint L_hip_x: limit lower=-0.523 upper=2.093 effort=60 velocity=0 -> lower=-0.523 upper=2.093 effort=100 velocity=10
- joint L_hip_y: limit lower=-3.14 upper=3.14 effort=120 velocity=0 -> lower=-3.14 upper=3.14 effort=250 velocity=10
- joint L_hip_z: limit lower=-3.14 upper=3.14 effort=60 velocity=0 -> lower=-3.14 upper=3.14 effort=100 velocity=10
- joint L_knee: limit lower=-1.919 upper=1.919 effort=120 velocity=0 -> lower=-1.919 upper=1.919 effort=250 velocity=10
- joint L_shoulder_x: type revolute -> fixed
- joint L_shoulder_y: type revolute -> fixed
- joint L_shoulder_z: type revolute -> fixed
- joint R_ankle_y: limit lower=-0.698 upper=0.698 effort=17 velocity=0 -> lower=-0.698 upper=0.698 effort=17 velocity=10
- joint R_elbow_x: type revolute -> fixed
- joint R_hip_x: limit lower=-2.093 upper=0.523 effort=60 velocity=0 -> lower=-2.093 upper=0.523 effort=100 velocity=10
- joint R_hip_y: limit lower=-3.14 upper=3.14 effort=120 velocity=0 -> lower=-3.14 upper=3.14 effort=250 velocity=10
- joint R_hip_z: limit lower=-3.14 upper=3.14 effort=60 velocity=0 -> lower=-3.14 upper=3.14 effort=100 velocity=10
- joint R_knee: limit lower=-1.919 upper=1.919 effort=120 velocity=0 -> lower=-1.919 upper=1.919 effort=250 velocity=10
- joint R_shoulder_x: type revolute -> fixed
- joint R_shoulder_y: type revolute -> fixed
- joint R_shoulder_z: type revolute -> fixed

Commit message: remove mujoco autoconvert (#10)
* remove mujoco autoconvert

* improve styling

* better options

* types

* fix static checks

* better test

* parse colors

* lint

File: tests/sample/robot.urdf (robot description, URDF)
Before this commit: robot robot, 20 links, 19 joints
Links:
- removed link L_buttock
- removed link L_calf
- removed link L_clav
- removed link L_farm
- removed link L_foot
- removed link L_leg
- removed link L_scapula
- removed link L_thigh
- removed link L_uarm
- removed link R_buttock
- removed link R_calf
- removed link R_clav
- removed link R_farm
- removed link R_foot
- removed link R_leg
- removed link R_scapula
- removed link R_thigh
- removed link R_uarm
- removed link base
- removed link trunk
- added link BODY, mass 27; visual box size=0.05 0.05 0.111; visual box size=0.08 0.08 0.08
- added link LARM_LINK1, mass 3; visual cylinder length=0.05 radius=0.025
- added link LARM_LINK2, mass 0.6; visual box size=0.05 0.05 0.163; visual cylinder length=0.05 radius=0.025
- added link LARM_LINK3, mass 1; visual cylinder length=0.05 radius=0.025
- added link LARM_LINK4, mass 0.6; visual box size=0.05 0.05 0.147; visual cylinder length=0.05 radius=0.025
- added link LARM_LINK5, mass 0.4; visual cylinder length=0.05 radius=0.025
- added link LARM_LINK6, mass 0.4; visual box size=0.05 0.03 0.175; visual cylinder length=0.05 radius=0.025
- added link LLEG_LINK1, mass 2.5; visual cylinder length=0.1 radius=0.05
- added link LLEG_LINK2, mass 2; visual cylinder length=0.1 radius=0.05
- added link LLEG_LINK3, mass 5.1; visual box size=0.1 0.1 0.1535; visual cylinder length=0.1 radius=0.05
- added link LLEG_LINK4, mass 7; visual box size=0.1 0.1 0.2; visual cylinder length=0.1 radius=0.05
- added link LLEG_LINK5, mass 2.5; visual cylinder length=0.1 radius=0.05
- added link RARM_LINK1, mass 3; visual cylinder length=0.05 radius=0.025
- added link RARM_LINK2, mass 0.6; visual box size=0.05 0.05 0.163; visual cylinder length=0.05 radius=0.025
- added link RARM_LINK3, mass 1; visual cylinder length=0.05 radius=0.025
- added link RARM_LINK4, mass 0.6; visual box size=0.05 0.05 0.147; visual cylinder length=0.05 radius=0.025
- added link RARM_LINK5, mass 0.4; visual cylinder length=0.05 radius=0.025
- added link RARM_LINK6, mass 0.4; visual box size=0.05 0.03 0.175; visual cylinder length=0.05 radius=0.025
- added link RLEG_LINK1, mass 2.5; visual cylinder length=0.1 radius=0.05
- added link RLEG_LINK2, mass 2; visual cylinder length=0.1 radius=0.05
- added link RLEG_LINK3, mass 5.1; visual box size=0.1 0.1 0.1535; visual cylinder length=0.1 radius=0.05
- added link RLEG_LINK4, mass 7; visual box size=0.1 0.1 0.2; visual cylinder length=0.1 radius=0.05
- added link RLEG_LINK5, mass 2.5; visual cylinder length=0.1 radius=0.05
- added link WAIST_LINK1, mass 6; visual cylinder length=0.05 radius=0.025
- added link WAIST_LINK2, mass 30; visual box size=0.05 0.05 0.275; visual cylinder length=0.05 radius=0.025
- added link base_link
- added link l_ankle, mass 1.9; visual box size=0.25 0.14 0.02; visual cylinder length=0.1 radius=0.05
- added link l_wrist, mass 0.4; visual box size=0.05 0.03 0.15
- added link r_ankle, mass 1.9; visual box size=0.25 0.14 0.02; visual cylinder length=0.1 radius=0.05
- added link r_wrist, mass 0.4; visual box size=0.05 0.03 0.15
- added link torso, mass 13; visual box size=0.05 0.05 0.03; visual box size=0.15 0.27 0.05
Joints:
- removed joint L_ankle_y
- removed joint L_elbow_x
- removed joint L_hip_x
- removed joint L_hip_y
- removed joint L_hip_z
- removed joint L_knee
- removed joint L_shoulder_x
- removed joint L_shoulder_y
- removed joint L_shoulder_z
- removed joint R_ankle_y
- removed joint R_elbow_x
- removed joint R_hip_x
- removed joint R_hip_y
- removed joint R_hip_z
- removed joint R_knee
- removed joint R_shoulder_x
- removed joint R_shoulder_y
- removed joint R_shoulder_z
- removed joint floating_base
- added joint CHEST: type revolute, parent WAIST_LINK2, child torso, origin xyz=0 0 0.35 rpy=0 0 0, axis 0 0 1, limit lower=-1.27 upper=1.27 effort=30 velocity=1.76
- added joint LARM_ELBOW: type revolute, parent LARM_LINK3, child LARM_LINK4, origin xyz=0 0 0 rpy=0 0 0, axis 0 1 0, limit lower=-2.42600766027 upper=2.42600766027 effort=70.0 velocity=4.58
- added joint LARM_SHOULDER_P: type revolute, parent torso, child LARM_LINK1, origin xyz=0 0.21 0 rpy=0 0 0, axis 0 1 0, limit lower=-1.57079632679 upper=0.785398163397 effort=100.0 velocity=2.7
- added joint LARM_SHOULDER_R: type revolute, parent LARM_LINK1, child LARM_LINK2, origin xyz=0 0 0 rpy=0 0 0, axis 1 0 0, limit lower=0.00872664625997 upper=2.87106661953 effort=100.0 velocity=3.66
- added joint LARM_SHOULDER_Y: type revolute, parent LARM_LINK2, child LARM_LINK3, origin xyz=0 0 -0.263 rpy=0 0 0, axis 0 0 1, limit lower=-1.57079632679 upper=0.785398163397 effort=100.0 velocity=2.7
- added joint LARM_WRIST_P: type revolute, parent LARM_LINK5, child LARM_LINK6, origin xyz=0 0 0 rpy=0 0 0, axis 0 1 0, limit lower=-2.51327412287 upper=2.51327412287 effort=20.0 velocity=1.95
- added joint LARM_WRIST_R: type revolute, parent LARM_LINK6, child l_wrist, origin xyz=0 0 0 rpy=0 0 0, axis 1 0 0, limit lower=-1.37008346282 upper=1.37008346282 effort=8.0 velocity=1.76
- added joint LARM_WRIST_Y: type revolute, parent LARM_LINK4, child LARM_LINK5, origin xyz=0 0 -0.247 rpy=0 0 0, axis 0 0 1, limit lower=-2.23402144255 upper=0.00349065850399 effort=70.0 velocity=4.58
- added joint LLEG_ANKLE_P: type revolute, parent LLEG_LINK4, child LLEG_LINK5, origin xyz=0 0 -0.3 rpy=0 0 0, axis 0 1 0, limit lower=0 upper=2.618 effort=300 velocity=7
- added joint LLEG_ANKLE_R: type revolute, parent LLEG_LINK5, child l_ankle, origin xyz=0 0 0 rpy=0 0 0, axis 1 0 0, limit lower=-1.27 upper=0.68 effort=160 velocity=5.8
- added joint LLEG_HIP_P: type revolute, parent LLEG_LINK1, child LLEG_LINK2, origin xyz=0 0 0 rpy=0 0 0, axis 0 1 0, limit lower=-0.349065850399 upper=1.57079632679 effort=100 velocity=3.87
- added joint LLEG_HIP_R: type revolute, parent BODY, child LLEG_LINK1, origin xyz=0 0.09 0 rpy=0 0 0, axis 1 0 0, limit lower=-0.349065850399 upper=1.57079632679 effort=100 velocity=3.87
- added joint LLEG_HIP_Y: type revolute, parent LLEG_LINK2, child LLEG_LINK3, origin xyz=0 0 -0.3535 rpy=0 0 0, axis 0 0 1, limit lower=-0.5236 upper=0.5236 effort=160 velocity=5.8
- added joint LLEG_KNEE: type revolute, parent LLEG_LINK3, child LLEG_LINK4, origin xyz=0 0 0 rpy=0 0 0, axis 0 1 0, limit lower=-2.095 upper=0.7 effort=160 velocity=5.8
- added joint RARM_ELBOW: type revolute, parent RARM_LINK3, child RARM_LINK4, origin xyz=0 0 0 rpy=0 0 0, axis 0 1 0, limit lower=-2.23402144255 upper=0.00349065850399 effort=70.0 velocity=4.58
- added joint RARM_SHOULDER_P: type revolute, parent torso, child RARM_LINK1, origin xyz=0 -0.21 0 rpy=0 0 0, axis 0 1 0, limit lower=-1.57079632679 upper=0.785398163397 effort=100.0 velocity=2.7
- added joint RARM_SHOULDER_R: type revolute, parent RARM_LINK1, child RARM_LINK2, origin xyz=0 0 0 rpy=0 0 0, axis 1 0 0, limit lower=0.00872664625997 upper=2.87106661953 effort=100.0 velocity=3.66
- added joint RARM_SHOULDER_Y: type revolute, parent RARM_LINK2, child RARM_LINK3, origin xyz=0 0 -0.263 rpy=0 0 0, axis 0 0 1, limit lower=-2.42600766027 upper=2.42600766027 effort=70.0 velocity=4.58
- added joint RARM_WRIST_P: type revolute, parent RARM_LINK5, child RARM_LINK6, origin xyz=0 0 0 rpy=0 0 0, axis 0 1 0, limit lower=-1.37008346282 upper=1.37008346282 effort=8.0 velocity=1.76
- added joint RARM_WRIST_R: type revolute, parent RARM_LINK6, child r_wrist, origin xyz=0 0 0 rpy=0 0 0, axis 1 0 0, limit lower=-0.680678408278 upper=0.680678408278 effort=8.0 velocity=1.76
- added joint RARM_WRIST_Y: type revolute, parent RARM_LINK4, child RARM_LINK5, origin xyz=0 0 -0.247 rpy=0 0 0, axis 0 0 1, limit lower=-2.51327412287 upper=2.51327412287 effort=20.0 velocity=1.95
- added joint RLEG_ANKLE_P: type revolute, parent RLEG_LINK4, child RLEG_LINK5, origin xyz=0 0 -0.3 rpy=0 0 0, axis 0 1 0, limit lower=0 upper=2.618 effort=30 velocity=5.8
- added joint RLEG_ANKLE_R: type revolute, parent RLEG_LINK5, child r_ankle, origin xyz=0 0 0 rpy=0 0 0, axis 1 0 0, limit lower=-1.27 upper=0.68 effort=160 velocity=5.8
- added joint RLEG_HIP_P: type revolute, parent RLEG_LINK1, child RLEG_LINK2, origin xyz=0 0 0 rpy=0 0 0, axis 0 1 0, limit lower=-0.5236 upper=0.5236 effort=160 velocity=5.8
- added joint RLEG_HIP_R: type revolute, parent BODY, child RLEG_LINK1, origin xyz=0 -0.09 0 rpy=0 0 0, axis 1 0 0, limit lower=-0.349065850399 upper=1.57079632679 effort=100 velocity=3.87
- added joint RLEG_HIP_Y: type revolute, parent RLEG_LINK2, child RLEG_LINK3, origin xyz=0 0 -0.3535 rpy=0 0 0, axis 0 0 1, limit lower=-2.095 upper=0.7 effort=160 velocity=5.8
- added joint RLEG_KNEE: type revolute, parent RLEG_LINK3, child RLEG_LINK4, origin xyz=0 0 0 rpy=0 0 0, axis 0 1 0, limit lower=0 upper=2.618 effort=300 velocity=7
- added joint WAIST_P: type revolute, parent BODY, child WAIST_LINK1, origin xyz=0 0 0.176 rpy=0 0 0, axis 0 1 0, limit lower=-1.27 upper=1.27 effort=30 velocity=1.76
- added joint WAIST_R: type revolute, parent WAIST_LINK1, child WAIST_LINK2, origin xyz=0 0 0 rpy=0 0 0, axis 1 0 0, limit lower=-1.27 upper=1.27 effort=30 velocity=1.76
- added joint waist: type fixed, parent base_link, child BODY, origin xyz=0 0 0 rpy=0 0 0

Commit message: more options (#17)
* more options

* fix cli

* fix tests

File: tests/sample/robot.urdf (robot description, URDF)
Before this commit: robot simple_humanoid, 31 links, 30 joints
Links:
- added link IMU, mass 0; visual box size=0.05 0.05 0.05
Joints:
- added joint imu: type fixed, parent BODY, child IMU, origin xyz=0 0 0 rpy=0 0 0

Commit message: better joint simplification (#23)
* better joint simplification

* fix test

File: tests/sample/robot.urdf (robot description, URDF)
Before this commit: robot simple_humanoid, 32 links, 31 joints
Links:
- removed link base_link
Joints:
- removed joint waist

Commit message: Backlash (#48)
* backlash

* backlash implementation

* add floor pass

File: tests/sample/robot.urdf (robot description, URDF)
Before this commit: robot simple_humanoid, 31 links, 30 joints
Links:
- link l_ankle: geometry collision box size=0.25 0.14 0.02; visual box size=0.25 0.14 0.02
- link r_ankle: geometry collision box size=0.25 0.14 0.02; visual box size=0.25 0.14 0.02
